File: KiCad/HB15.sch (KiCad schematic (older format))
At the start: 73 parts, among them J1 1964, J2 1966, SW1 SW_DPST_x2, SW2 SW_DPST_x2

Commit message: v2 before KiCad6 to rebase with the final commit
Parts:
- added R26: 10k 1W, symbol Device:R
- C20: value 100nF 400V POLY -> 100nF 400V
- SVolume: value A50k -> A1M
- renumbered SW1 to Boost64-, SW2 to Boost66-, R26 to R27, R27 to R28, R28 to R29, R29 to R30, R30 to R31, R31 to R32, R32 to R33, R33 to R34
Connections:
- net B+4a: now also R11.2, R17.2, R7.2, R8.2; no longer R32.2, V3.1 (A)
- net B+4b: now also R32.2, R26.1; no longer R11.2, R17.2, R7.2, R8.2
- new net: R26.2, V3.1 (A)
Other:
- note added: "(1.35V)"
- note added: "(1.3V)"
- note added: "(1.58V)"
- note added: "(1.5V)"
- note added: "(108V)"
- note added: "(112V)"
- note added: "(143V)"
- note added: "(191V)"
- note added: "(2.27V)"
- note added: "(211V)"
- note added: "(248V)"
- note added: "(49V)"
- note added: "(62V)"
- note added: "(98V)"
- note added: "B-15NC"
- note added: "B-15NF"
- note added: "Drop voltage\nKeep anode safe\n300V to 280V"
- note added: "POLY"
Changed lines of the file:
@@
 Rev "1.0"
 Comp "https://github.com/mdouchement/Ampeg-HB15"
-Comment1 "Ampeg Heritage B15 with custom mods"
-Comment2 ""
-Comment3 ""
-Comment4 ""
+Comment1 "All resistors are 1/2W unless otherwise specified"
+Comment2 "(1964 bias setting voltages shown in parenthesis)"
+Comment3 "D.C. voltage reading with no signal inserted"
+Comment4 "Ampeg Heritage B15 with custom mods"
 $EndDescr
 $Comp
@@
 $EndComp
 $Comp
-L Switch:SW_DPST_x2 SW1
+L Switch:SW_DPST_x2 Boost64-
 U 1 1 618A445D
 P 1775 2825
-F 0 "SW1" H 1775 2968 50  0000 C CNN
+F 0 "Boost64-" H 1775 2968 50  0000 C CNN
 F 1 "SW_DPST_x2" H 1775 2969 50  0001 C CNN
 F 2 "" H 1775 2825 50  0001 C CNN
@@
 	2025 3200 2025 3250
 $Comp
-L Switch:SW_DPST_x2 SW1
+L Switch:SW_DPST_x2 Boost64-
 U 2 1 618CEFF8
 P 4650 2725
-F 0 "SW1" H 4650 2868 50  0000 C CNN
+F 0 "Boost64-" H 4650 2868 50  0000 C CNN
 F 1 "SW_DPST_x2" H 4650 2869 50  0001 C CNN
 F 2 "" H 4650 2725 50  0001 C CNN
@@
 	4375 2725 4375 2775
 $Comp
-L Switch:SW_DPST_x2 SW2
+L Switch:SW_DPST_x2 Boost66-
 U 1 1 618EC2B7
 P 1725 6475
-F 0 "SW2" H 1725 6618 50  0000 C CNN
+F 0 "Boost66-" H 1725 6618 50  0000 C CNN
 F 1 "SW_DPST_x2" H 1725 6619 50  0001 C CNN
 F 2 "" H 1725 6475 50  0001 C CNN
@@
 Connection ~ 1475 6475
 $Comp
-L Switch:SW_DPST_x2 SW2
+L Switch:SW_DPST_x2 Boost66-
 U 2 1 61901C9E
 P 3225 6425
-F 0 "SW2" H 3225 6568 50  0000 C CNN
+F 0 "Boost66-" H 3225 6568 50  0000 C CNN
 F 1 "SW_DPST_x2" H 3225 6569 50  0001 C CNN
 F 2 "" H 3225 6425 50  0001 C CNN
@@
 	8450 4350 8475 4350
 $Comp
-L Device:R R29
+L Device:R R30
 U 1 1 6189C297
 P 8675 5275
-F 0 "R29" V 8468 5275 50  0000 C CNN
+F 0 "R30" V 8468 5275 50  0000 C CNN
 F 1 "47k" V 8559 5275 50  0000 C CNN
 F 2 "" V 8605 5275 50  0001 C CNN
@@
 $EndComp
 $Comp
-L Device:R R28
+L Device:R R29
 U 1 1 618AD902
 P 8475 5475
-F 0 "R28" H 8405 5429 50  0000 R CNN
+F 0 "R29" H 8405 5429 50  0000 R CNN
 F 1 "1M" H 8405 5520 50  0000 R CNN
 F 2 "" V 8405 5475 50  0001 C CNN
@@
 $EndComp
 $Comp
-L Device:R R30
+L Device:R R31
 U 1 1 618C9D2E
 P 9075 5975
-F 0 "R30" H 9005 5929 50  0000 R CNN
+F 0 "R31" H 9005 5929 50  0000 R CNN
 F 1 "1k 1W" H 9005 6020 50  0000 R CNN
 F 2 "" V 9005 5975 50  0001 C CNN
@@
 	9075 5775 9500 5775
 $Comp
-L Device:R R31
+L Device:R R32
 U 1 1 618D8F7E
 P 9175 3625
-F 0 "R31" H 9105 3579 50  0000 R CNN
+F 0 "R32" H 9105 3579 50  0000 R CNN
 F 1 "100k 1W" H 9105 3670 50  0000 R CNN
 F 2 "" V 9105 3625 50  0001 C CNN
@@
 Wire Wire Line
 	3500 2025 3550 2025
-Wire Wire Line
-	8375 3100 8375 3225
 Text GLabel 8375 3100 1    50   Input ~ 0
+B+4b
+Text GLabel 3025 900  1    50   Input ~ 0
 B+4a
-Text GLabel 3025 900  1    50   Input ~ 0
-B+4b
 Text GLabel 2375 4500 1    50   Input ~ 0
-B+4b
+B+4a
 Wire Wire Line
 	4900 2725 4900 2775
@@
 $EndComp
 $Comp
-L Device:R R26
+L Device:R R27
 U 1 1 619B8100
 P 7975 4450
-F 0 "R26" H 7905 4404 50  0000 R CNN
+F 0 "R27" H 7905 4404 50  0000 R CNN
 F 1 "1M" H 7905 4495 50  0000 R CNN
 F 2 "" V 7905 4450 50  0001 C CNN
@@
 	7975 4250 7975 4300
 $Comp
-L Device:R R27
+L Device:R R28
 U 1 1 619C9618
 P 8150 4250
-F 0 "R27" V 7943 4250 50  0000 C CNN
+F 0 "R28" V 7943 4250 50  0000 C CNN
 F 1 "100" V 8034 4250 50  0000 C CNN
 F 2 "" V 8080 4250 50  0001 C CNN
@@
 P 5975 3750
 F 0 "SVolume" H 5906 3796 50  0000 R CNN
-F 1 "A50k" H 5906 3705 50  0000 R CNN
+F 1 "A1M" H 5906 3705 50  0000 R CNN
 F 2 "" H 5975 3750 50  0001 C CNN
 F 3 "~" H 5975 3750 50  0001 C CNN
@@
 Wire Wire Line
 	6125 3750 6150 3750
-Wire Wire Line
-	6875 3225 8375 3225
 $Comp
 L Device:C C20
@@
 P 7475 4650
 F 0 "C20" V 7223 4650 50  0000 C CNN
-F 1 "100nF 400V POLY" V 7314 4650 50  0000 C CNN
+F 1 "100nF 400V" V 7314 4650 50  0000 C CNN
 F 2 "" H 7513 4500 50  0001 C CNN
 F 3 "~" H 7475 4650 50  0001 C CNN
@@
 Wire Wire Line
 	9175 3225 9175 3475
-Connection ~ 8375 3225
 Wire Wire Line
 	9675 4650 9675 4700
@@
 $EndComp
 $Comp
-L Device:R R32
+L Device:R R33
 U 1 1 61A7B311
 P 9675 4500
-F 0 "R32" H 9605 4454 50  0000 R CNN
+F 0 "R33" H 9605 4454 50  0000 R CNN
 F 1 "1M" H 9605 4545 50  0000 R CNN
 F 2 "" V 9605 4500 50  0001 C CNN
@@
 $EndComp
 $Comp
-L Device:R R33
+L Device:R R34
 U 1 1 61A84A40
 P 9925 4200
-F 0 "R33" V 9718 4200 50  0000 C CNN
+F 0 "R34" V 9718 4200 50  0000 C CNN
 F 1 "47k" V 9809 4200 50  0000 C CNN
 F 2 "" V 9855 4200 50  0001 C CNN
@@
 Wire Wire Line
 	5500 3500 5500 4550
+Text Notes 7375 4825 0    50   ~ 0
+POLY
+$Comp
+L Device:R R26
+U 1 1 61916258
+P 7700 3225
+F 0 "R26" V 7493 3225 50  0000 C CNN
+F 1 "10k 1W" V 7584 3225 50  0000 C CNN
+F 2 "" V 7630 3225 50  0001 C CNN
+F 3 "~" H 7700 3225 50  0001 C CNN
+	1    7700 3225
+	0    1    1    0
+$EndComp
+Wire Wire Line
+	8375 3100 8375 3225
+Wire Wire Line
+	7850 3225 8375 3225
+Connection ~ 8375 3225
+Wire Wire Line
+	7550 3225 6875 3225
+Text Notes 7450 3525 0    50   ~ 0
+Drop voltage\nKeep anode safe\n300V to 280V
+Text Notes 6850 3175 0    50   ~ 0
+(191V)
+Text Notes 8450 3050 0    50   ~ 0
+(211V)
+Text Notes 9200 4825 0    50   ~ 0
+(62V)
+Text Notes 6900 4125 0    50   ~ 0
+(49V)
+Text Notes 9325 5625 0    50   ~ 0
+(1.5V)
+Text Notes 3100 875  0    50   ~ 0
+(248V)
+Text Notes 2475 4475 0    50   ~ 0
+(248V)
+Text Notes 1275 1800 0    50   ~ 0
+(108V)
+Text Notes 4125 1775 0    50   ~ 0
+(143V)
+Text Notes 4050 2825 0    50   ~ 0
+(2.27V)
+Text Notes 1250 2900 0    50   ~ 0
+(1.35V)
+Text Notes 1225 5575 0    50   ~ 0
+(98V)
+Text Notes 3175 5525 0    50   ~ 0
+(112V)
+Text Notes 2650 6475 0    50   ~ 0
+(1.3V)
+Text Notes 1325 6450 0    50   ~ 0
+(1.58V)
+Text Notes 500  5775 0    50   ~ 0
+B-15NF
+Text Notes 500  2125 0    50   ~ 0
+B-15NC
 $EndSCHEMATC
