File: KiCad/HB15.kicad_sch (KiCad schematic)
At the start: 74 parts, among them J1 1964, J2 1966

Commit message: v2
Parts:
- added BassX, TrebleX: A1M, symbol Device:R_POT
- added Both: SW_SPST, symbol Switch:SW_SPST
- added C900: 1nF, symbol Device:C
- added C901: 10nF, symbol Device:C
- added C902: 470pF, symbol Device:C
- added C903: 4.7nF, symbol Device:C
- added C904: 2.2nF, symbol Device:C
- added C905: 1.5nF, symbol Device:C
- added MidBoost (x2): SW_SPDT, symbol Switch:SW_SPDT
- added R900: 220k, symbol Device:R
- added R901: 22k, symbol Device:R
- added R902: 270k, symbol Device:R
- added R903: 120k, symbol Device:R
- added R904, R906: 1k, symbol Device:R
- added R905: 100k, symbol Device:R
- R34: value 47k -> 100k
Connections:
- net GND: now also C10.1, C17.1, C904.1, C905.1, MidBoost.1 (A), MidBoost.1 (A), R902.1, R905.1; no longer C10.2, C17.2
- net at J1.T, R2.2: now also Both.1 (A)
- net at C3.1, C9.2: now also R12.2; no longer R12.1
- net at Bass64.3, C6.2: now also R12.1; no longer R12.2
- net at Bass64.2, C6.1, R13.2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: now also C7.1; no longer C7.2
- net at Bass64.1, R14.2: now also C7.2; no longer C7.1
- net at Treble64.1: now also C10.2; no longer C10.1
- net at J2.T, R1.2: now also Both.2 (B)
- net at C11.1, C16.2: now also R18.2; no longer R18.1
- net at Bass66.2, C12.1, R15.2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: now also C13.1; no longer C13.2
- net at Treble66.1: now also C17.2; no longer C17.1
- net at Bass66.1, R20.2: now also C13.2; no longer C13.1
- net at Bass66.3, C12.2: now also R18.1; no longer R18.2
- net B+4a renamed B+4ps
- net B+4b renamed B+4el
- new net: BassX.2, C900.1, C901.1, R902.2, R903.2
- new net: C904.2, MidBoost.3 (C), R904.2
- new net: C903.2, TrebleX.1
- new net: C902.1, TrebleX.3
- new net: C903.1, MidBoost.2 (B)
- new net: C905.2, MidBoost.3 (C), R906.1
- new net: MidBoost.2 (B), R901.1
- new net: BassX.1, C901.2, R901.2
- new net: BassX.3, C900.2, R900.1
- new net: R904.1, R905.2, R906.2
- new net IN: C902.2, R900.2
- new net OUT: R903.1, TrebleX.2
Other:
- note added: "1.6V (1.6V)"
- note added: "1.9V (1.9V)"
- note added: "106V (106V)"
- note added: "144V (146V)"
- note added: "150V (151V)"
- note added: "152V (152V)"
- note added: "2.6V (2.6V)"
- note added: "204V (206V)"
- note added: "237V (236V)"
- note added: "264V (264V)"
- note added: "310V (310V)"
- note added: "63V (63V)"
- note added: "Drop voltage to keep anode safe B+4el may go over 300VDC depending the electrical grid fluctuation"
- note added: "Mid boost mod implementation example"
- note removed: "(1.35V)"
- note removed: "(1.3V)"
- note removed: "(1.58V)"
- note removed: "(1.5V)"
- note removed: "(108V)"
- note removed: "(112V)"
- note removed: "(143V)"
- note removed: "(191V)"
- note removed: "(2.27V)"
- note removed: "(211V)"
- note removed: "(248V)"
- note removed: "(49V)"
- note removed: "(62V)"
- note removed: "(98V)"
- note removed: "Drop voltage Keep anode safe 300V to 280V"
- moved on the sheet: Boost64-A, Boost64-B, Boost66-A, Boost66-B, Bright, C1, C11, C14, C15, C18, C19, C2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
