File: KiCad/Power.kicad_sch (KiCad schematic)
At the start: 69 parts, among them J3 Conn_IEC-320-C13_Socket, T1 373BX, T2 1650PA

Commit message: v2
Parts:
- added NFB_: ON-OFF-ON, symbol Switch:SW_DPDT_x2
- added R60: 10k 1W, symbol Device:R
- R40: value 22k 2W -> 10k 2W
Connections:
- net at R39.1, V4.3 (K): now also NFB_.2 (B); no longer R52.2
- net at R52.1: now also NFB_.3 (C), NFB_.4 (A); no longer T2.4Ω (GRN)
- net at T1.120V (BLU): now also OFF-STANDBY-ON-.3 (C); no longer T1.0V (YEL/BLK)
- net B+4a renamed B+4el
- net B+4b renamed B+4ps
- new net: NFB_.1 (A), R52.2, R60.2
- new net: T1.0V (YEL/BLK), T1.120V (BLU)
- new net: NFB_.5 (B), T2.4Ω (GRN)
- new net: NFB_.6 (C), R60.1
- now unconnected: T1.110V (BLU/YEL)
Other:
- note added: "-41V"
- note added: "-41V (0V)"
- note added: "0V (36V)"
- note added: "1.9V (1.9V)"
- note added: "204V (203V)"
- note added: "212V (210V)"
- note added: "230VAC"
- note added: "264V (264V)"
- note added: "2V (2V)"
- note added: "310V (310V)"
- note added: "351V (354V)"
- note added: "360V (360V)"
- note added: "373BX is wired in 240VAC on a 230VAC electrical grid. It allows to reduce B+ to ~450VDC. Heaters remains at a voltage above 6.3VCT."
- note added: "444V (440V)"
- note added: "448V (448V)"
- note added: "450V (451V)"
- note added: "452V (453V)"
- note added: "on: Original 3.3k NFB but with rumble at high volume off: Disabled NFB to get a different voicing on: Custom 13.3k stable NFB at high volume"
- note removed: "(0V)"
- note removed: "(1.69V)"
- note removed: "(1.6V)"
- note removed: "(157V)"
- note removed: "(165V)"
- note removed: "(211V)"
- note removed: "(248V)"
- note removed: "(294V)"
- note removed: "(36.6V)"
- note removed: "(360V)"
- note removed: "(454V)"
- note removed: "(464V)"
- note removed: "(469V)"
- note removed: "(470V)"
- note removed: "0V"
- note removed: "230V"
- moved on the sheet: OFF-STANDBY-ON-A, R52
